Commit message: Structure: Move motor_node and esp32_encoder to correct path, update xacro descriptions

File: src/my_bot/description/lidar.xacro (robot description, xacro)
@@ -2,21 +2,21 @@
 <robot xmlns:xacro="http://www.ros.org/wiki/xacro" >
     <joint name="laser_joint" type="fixed">
-        <parent link="chassis"/>
+        <parent link="base_link"/>
         <child link="laser_frame"/>
-        <origin xyz="0.075 0 0.125" rpy="0 0 0"/>
+        <origin xyz="-0.035 0 0.125" rpy="0 0 0"/>
     </joint>
     <link name="laser_frame">
         <visual>
             <geometry>
-                <cylinder radius="0.035" length="0.025"/>
+                <cylinder radius="0.03" length="0.015"/>
             </geometry>
-            <material name="whilte"/>
+            <material name="white"/>
         </visual>
         <collision>
             <geometry>
-                <cylinder radius="0.035" length="0.025"/>
+                <cylinder radius="0.03" length="0.015"/>
             </geometry>
         </collision>
-        <xacro:inertial_cylinder mass="0.1" length="0.025" radius="0.035">
+        <xacro:inertial_cylinder mass="0.1" length="0.015" radius="0.03">
             <origin xyz="0 0 0" rpy="0 0 0"/>
         </xacro:inertial_cylinder>

File: src/my_bot/description/robot_core.xacro (robot description, xacro)
@@ -18,11 +18,4 @@
     </material>
     <link name="base_link">
-    </link>
-    <joint name="base_footprint_joint" type="fixed">
-        <parent link="base_link"/>
-        <child link="base_footprint"/>
-        <origin xyz="0 0 0" rpy="0 0 0"/>
-    </joint>
-    <link name="base_footprint">
     </link>
     <joint name="chassis_joint" type="fixed">
@@ -146,18 +139,18 @@
     <link name="chassis_3">
         <visual>
-            <origin xyz="0.08 0 0.1" />
+            <origin xyz="0.07 0 0.1" />
             <geometry>
-                <box size="0.08 0.07 0.035"/>
+                <box size="0.08 0.06 0.035"/>
             </geometry>
             <material name="black"/>
         </visual>
         <collision>
-            <origin xyz="0.08 0 0.1" />
+            <origin xyz="0.07 0 0.1" />
             <geometry>
-                <box size="0.08 0.07 0.035"/>
+                <box size="0.08 0.06 0.035"/>
             </geometry>
         </collision>
-        <xacro:inertial_box mass="0.2" x="0.08" y="0.07" z="0.035">
-            <origin xyz="0.08 0 0.0825" rpy="0 0 0" /> </xacro:inertial_box>
+        <xacro:inertial_box mass="0.2" x="0.08" y="0.06" z="0.035">
+            <origin xyz="0.07 0 0.1" rpy="0 0 0" /> </xacro:inertial_box>
     </link>
     <gazebo reference="chassis_2">
